Commit message: Update backpack_3d.urdf

File: backpack_3d.urdf (robot description, URDF)
Before this commit: robot cartographer_backpack_3d, 3 links, 2 joints
Links:
- removed link horizontal_vlp16_link
- added link velodyne; visual cylinder length=0.07 radius=0.05
Joints:
- removed joint horizontal_vlp16_link_joint
- added joint velodyne_joint: type fixed, parent base_link, child velodyne, origin xyz=0.01 0. 0.19 rpy=0. -0.1745 3.1416
